Commit message: Added asteroid generator, Added Gazebo launch file, Fixed package naming convention

File: arm_game/urdf/kr16_2.urdf (robot description, URDF)
Before this commit: robot kuka_kr16_2, 10 links, 9 joints
Links:
- link base_link: geometry collision mesh filename=package://arm_game/meshes/kr16_2/collision/base_link.stl; visual mesh filename=package://arm_game/meshes/kr16_2/visual/base_link.dae
- link link_1: geometry collision mesh filename=package://arm_game/meshes/kr16_2/collision/link_1.stl; visual mesh filename=package://arm_game/meshes/kr16_2/visual/link_1.dae
- link link_2: geometry collision mesh filename=package://arm_game/meshes/kr16_2/collision/link_2.stl; visual mesh filename=package://arm_game/meshes/kr16_2/visual/link_2.dae
- link link_3: geometry collision mesh filename=package://arm_game/meshes/kr16_2/collision/link_3.stl; visual mesh filename=package://arm_game/meshes/kr16_2/visual/link_3.dae
- link link_4: geometry collision mesh filename=package://arm_game/meshes/kr16_2/collision/link_4.stl; visual mesh filename=package://arm_game/meshes/kr16_2/visual/link_4.dae
- link link_5: geometry collision mesh filename=package://arm_game/meshes/kr16_2/collision/link_5.stl; visual mesh filename=package://arm_game/meshes/kr16_2/visual/link_5.dae
- link link_6: geometry collision mesh filename=package://arm_game/meshes/kr16_2/collision/link_6.stl; visual mesh filename=package://arm_game/meshes/kr16_2/visual/link_6.dae

File: arm_game/urdf/kr210l150.urdf (robot description, URDF)
Before this commit: robot kuka_kr210, 10 links, 9 joints
Links:
- link base_link: geometry collision mesh filename=package://arm_game/meshes/kr210l150/collision/base_link.stl; visual mesh filename=package://arm_game/meshes/kr210l150/visual/base_link.dae
- link link_1: geometry collision mesh filename=package://arm_game/meshes/kr210l150/collision/link_1.stl; visual mesh filename=package://arm_game/meshes/kr210l150/visual/link_1.dae
- link link_2: geometry collision mesh filename=package://arm_game/meshes/kr210l150/collision/link_2.stl; visual mesh filename=package://arm_game/meshes/kr210l150/visual/link_2.dae
- link link_3: geometry collision mesh filename=package://arm_game/meshes/kr210l150/collision/link_3.stl; visual mesh filename=package://arm_game/meshes/kr210l150/visual/link_3.dae
- link link_4: geometry collision mesh filename=package://arm_game/meshes/kr210l150/collision/link_4.stl; visual mesh filename=package://arm_game/meshes/kr210l150/visual/link_4.dae
- link link_5: geometry collision mesh filename=package://arm_game/meshes/kr210l150/collision/link_5.stl; visual mesh filename=package://arm_game/meshes/kr210l150/visual/link_5.dae
- link link_6: geometry collision mesh filename=package://arm_game/meshes/kr210l150/collision/link_6.stl; visual mesh filename=package://arm_game/meshes/kr210l150/visual/link_6.dae

File: arm_game/urdf/kuka.urdf (robot description, URDF)
Before this commit: robot kuka_lbr_iiwa_14_r820, 11 links, 10 joints
Links:
- link base_link: geometry collision mesh filename=package://arm_game/meshes/lbr_iiwa_14_r820/collision/base_l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; visual mesh filename=package://arm_game/meshes/lbr_iiwa_14_r820/visual/base_link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
- link link_1: geometry collision mesh filename=package://arm_game/meshes/lbr_iiwa_14_r820/collision/link_1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; visual mesh filename=package://arm_game/meshes/lbr_iiwa_14_r820/visual/link_1.dae
- link link_2: geometry collision mesh filename=package://arm_game/meshes/lbr_iiwa_14_r820/collision/link_2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; visual mesh filename=package://arm_game/meshes/lbr_iiwa_14_r820/visual/link_2.dae
- link link_3: geometry collision mesh filename=package://arm_game/meshes/lbr_iiwa_14_r820/collision/link_3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; visual mesh filename=package://arm_game/meshes/lbr_iiwa_14_r820/visual/link_3.dae
- link link_4: geometry collision mesh filename=package://arm_game/meshes/lbr_iiwa_14_r820/collision/link_4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; visual mesh filename=package://arm_game/meshes/lbr_iiwa_14_r820/visual/link_4.dae
- link link_5: geometry collision mesh filename=package://arm_game/meshes/lbr_iiwa_14_r820/collision/link_5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; visual mesh filename=package://arm_game/meshes/lbr_iiwa_14_r820/visual/link_5.dae
- link link_6: geometry collision mesh filename=package://arm_game/meshes/lbr_iiwa_14_r820/collision/link_6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; visual mesh filename=package://arm_game/meshes/lbr_iiwa_14_r820/visual/link_6.dae
- link link_7: geometry collision mesh filename=package://arm_game/meshes/lbr_iiwa_14_r820/collision/link_7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; visual mesh filename=package://arm_game/meshes/lbr_iiwa_14_r820/visual/link_7.dae

File: arm_game/urdf/panda_arm.urdf (robot description, URDF)
Before this commit: robot panda, 9 links, 8 joints
Links:
- link panda_link0: geometry collision cylinder length=0.03 radius=0.09; collision sphere radius=0.09
- link panda_link1: geometry collision cylinder length=0.2830 radius=0.09; collision sphere radius=0.09
- link panda_link2: geometry collision cylinder length=0.12 radius=0.09; collision sphere radius=0.09
- link panda_link3: geometry collision cylinder length=0.15 radius=0.09; collision sphere radius=0.09
- link panda_link4: geometry collision cylinder length=0.12 radius=0.09; collision sphere radius=0.09
- link panda_link5: geometry collision cylinder length=0.1 radius=0.09; collision cylinder length=0.14 radius=0.055
- link panda_link6: geometry collision cylinder length=0.08 radius=0.08; collision sphere radius=0.08
- link panda_link7: geometry collision cylinder length=0.14 radius=0.07; collision sphere radius=0.07
