Commit message: First round of changes for urdf

File: arm_game/urdf/kuka.urdf (robot description, URDF)
Before this commit: robot kuka_lbr_iiwa_14_r820, 11 links, 10 joints
Links:
- removed link base
- removed link tool0
- link base_link: mass None -> 0
- link link_1: mass None -> 2.0
- link link_2: mass None -> 2.0
- link link_3: mass None -> 2.0
- link link_4: mass None -> 2.0
- link link_5: mass None -> 2.0
- link link_6: mass None -> 2.0
- link link_7: mass None -> 2.0
Joints:
- removed joint base_link-base
- removed joint joint_a7-tool0
- joint joint_a1: limit lower=-2.9668 upper=2.9668 effort=0 velocity=1.4834 -> lower=-2.96705972839 upper=2.96705972839 effort=204 velocity=1.91986217719; origin xyz=0 0 0 rpy=0 0 0 -> xyz=0 0 0.11 rpy=0 0 0
- joint joint_a2: axis 0 1 0 -> 0 -1 0; origin xyz=-0.00043624 0 0.36 rpy=0 0 0 -> xyz=0 0 0.20 rpy=0 0 0
- joint joint_a3: limit lower=-2.9668 upper=2.9668 effort=0 velocity=1.7452 -> lower=-2.96705972839 upper=2.96705972839 effort=204 velocity=2.26892802759; origin xyz=0 0 0 rpy=0 0 0 -> xyz=0 0 0.20 rpy=0 0 0
- joint joint_a4: axis 0 -1 0 -> 0 1 0; limit lower=-2.0942 upper=2.0942 effort=0 velocity=1.3089 -> lower=-2.09439510239 upper=2.09439510239 effort=306 velocity=2.26892802759; origin xyz=0.00043624 0 0.42 rpy=0 0 0 -> xyz=0 0 0.20 rpy=0 0 0
- joint joint_a5: limit lower=-2.9668 upper=2.9668 effort=0 velocity=2.2688 -> lower=-2.96705972839 upper=2.96705972839 effort=204 velocity=2.26892802759; origin xyz=0 0 0 rpy=0 0 0 -> xyz=0 0 0.20 rpy=0 0 0
- joint joint_a6: axis 0 1 0 -> 0 -1 0; limit lower=-2.0942 upper=2.0942 effort=0 velocity=2.356 -> lower=-2.09439510239 upper=2.09439510239 effort=306 velocity=3.14159265359; origin xyz=0 0 0.4 rpy=0 0 0 -> xyz=0 0 0.19 rpy=0 0 0
- joint joint_a7: limit lower=-3.0541 upper=3.0541 effort=0 velocity=2.356 -> lower=-2.96705972839 upper=2.96705972839 effort=204 velocity=3.14159265359; origin xyz=0 0 0 rpy=0 0 0 -> xyz=0 0 0.078 rpy=0 0 0

Commit message: Hey hey!! Gazebo works!

File: arm_game/urdf/kuka.urdf (robot description, URDF)
Before this commit: robot kuka, 9 links, 8 joints
Links:
- added link base
- added link tool0
- link base_link: mass 0 -> None
- link link_1: mass 2.0 -> None
- link link_2: mass 2.0 -> None
- link link_3: mass 2.0 -> None
- link link_4: mass 2.0 -> None
- link link_5: mass 2.0 -> None
- link link_6: mass 2.0 -> None
- link link_7: mass 2.0 -> None
Joints:
- added joint base_link-base: type fixed, parent base_link, child base, origin xyz=0 0 0 rpy=0 0 0
- added joint joint_a7-tool0: type fixed, parent link_7, child tool0, origin xyz=0 0 0.126 rpy=0 0 0, axis 0 0 0
- joint joint_a1: limit lower=-2.96705972839 upper=2.96705972839 effort=204 velocity=1.91986217719 -> lower=-2.9668 upper=2.9668 effort=0 velocity=1.4834; origin xyz=0 0 0.11 rpy=0 0 0 -> xyz=0 0 0 rpy=0 0 0
- joint joint_a2: axis 0 -1 0 -> 0 1 0; origin xyz=0 0 0.20 rpy=0 0 0 -> xyz=-0.00043624 0 0.36 rpy=0 0 0
- joint joint_a3: limit lower=-2.96705972839 upper=2.96705972839 effort=204 velocity=2.26892802759 -> lower=-2.9668 upper=2.9668 effort=0 velocity=1.7452; origin xyz=0 0 0.20 rpy=0 0 0 -> xyz=0 0 0 rpy=0 0 0
- joint joint_a4: axis 0 1 0 -> 0 -1 0; limit lower=-2.09439510239 upper=2.09439510239 effort=306 velocity=2.26892802759 -> lower=-2.0942 upper=2.0942 effort=0 velocity=1.3089; origin xyz=0 0 0.20 rpy=0 0 0 -> xyz=0.00043624 0 0.42 rpy=0 0 0
- joint joint_a5: limit lower=-2.96705972839 upper=2.96705972839 effort=204 velocity=2.26892802759 -> lower=-2.9668 upper=2.9668 effort=0 velocity=2.2688; origin xyz=0 0 0.20 rpy=0 0 0 -> xyz=0 0 0 rpy=0 0 0
- joint joint_a6: axis 0 -1 0 -> 0 1 0; limit lower=-2.09439510239 upper=2.09439510239 effort=306 velocity=3.14159265359 -> lower=-2.0942 upper=2.0942 effort=0 velocity=2.356; origin xyz=0 0 0.19 rpy=0 0 0 -> xyz=0 0 0.4 rpy=0 0 0
- joint joint_a7: limit lower=-2.96705972839 upper=2.96705972839 effort=204 velocity=3.14159265359 -> lower=-3.0541 upper=3.0541 effort=0 velocity=2.356; origin xyz=0 0 0.078 rpy=0 0 0 -> xyz=0 0 0 rpy=0 0 0
