Commit message: added in safety controller and dynamics for prismatic joints

File: arm_game/urdf/iiwa7_9dof.xacro (robot description, xacro)
@@ -2,7 +2,7 @@
 <robot xmlns:xacro="http://www.ros.org/wiki/xacro">
   <!-- Import all Gazebo-customization elements, including Gazebo colors -->
-  <xacro:include filename="$(find arm_game)/urdf/iiwa.gazebo.xacro" />
+  <xacro:include filename="$(find arm_game)/urdf/iiwa.gazebo_9dof.xacro" />
   <!-- Import Transmissions -->
-  <xacro:include filename="$(find arm_game)/urdf/iiwa.transmission.xacro" />
+  <xacro:include filename="$(find arm_game)/urdf/iiwa.transmission_9dof.xacro" />
   <!-- Include Utilities -->
   <xacro:include filename="$(find arm_game)/urdf/utilities.xacro" />
@@ -47,4 +47,9 @@
       <axis xyz="1 0 0"/>
       <limit  lower="-1"  upper="1" effort="100" velocity="10"/>
+      <safety_controller soft_lower_limit="${-173 / 180}"
+                         soft_upper_limit="${173 / 180}"
+                         k_position="${safety_controller_k_pos}"
+                         k_velocity="${safety_controller_k_vel}"/>
+      <dynamics damping="${joint_damping}"/>
     </joint>
     <link name="${robot_name}_link_0a">
@@ -62,4 +67,9 @@
       <axis xyz="0 1 0"/>
       <limit  lower="-1"  upper="1" effort="100" velocity="10"/>
+      <safety_controller soft_lower_limit="${-173 / 180}"
+                         soft_upper_limit="${173 / 180}"
+                         k_position="${safety_controller_k_pos}"
+                         k_velocity="${safety_controller_k_vel}"/>
+      <dynamics damping="${joint_damping}"/>
     </joint>
     <link name="${robot_name}_link_0b">
