Commit message: 9DOF loads in Gazebo

File: arm_game/urdf/iiwa.transmission_9dof.xacro (robot description, xacro)
@@ -20,4 +20,15 @@
       </joint>
       <actuator name="${robot_name}_motor_0y">
+	<hardwareInterface>${hardware_interface}</hardwareInterface>
+	<mechanicalReduction>1</mechanicalReduction>
+      </actuator>
+    </transmission>
+    <transmission name="${robot_name}_tran_1">
+      <robotNamespace>/${robot_name}</robotNamespace>
+      <type>transmission_interface/SimpleTransmission</type>
+      <joint name="${robot_name}_joint_1">
+	<hardwareInterface>${hardware_interface}</hardwareInterface>
+      </joint>
+      <actuator name="${robot_name}_motor_1">
 	<hardwareInterface>${hardware_interface}</hardwareInterface>
 	<mechanicalReduction>1</mechanicalReduction>
