Commit message: bucket color fixed

File: arm_game/urdf/iiwa.gazebo.xacro (robot description, xacro)
@@ -56,7 +56,7 @@
       <mu2>0.2</mu2>
     </gazebo>
-	    <!-- Bucket -->
+    <!-- Bucket -->
     <gazebo reference="${robot_name}_bucket">
-      <material>Gazebo/Grey</material>
+      <material>Gazebo/Red</material>
       <mu1>0.2</mu1>
       <mu2>0.2</mu2>

File: arm_game/urdf/iiwa.gazebo_9dof.xacro (robot description, xacro)
@@ -68,7 +68,7 @@
       <mu2>0.2</mu2>
     </gazebo>
-	    <!-- Bucket -->
+    <!-- Bucket -->
     <gazebo reference="${robot_name}_bucket">
-      <material>Gazebo/Grey</material>
+      <material>Gazebo/Red</material>
       <mu1>0.2</mu1>
       <mu2>0.2</mu2>
